File: vfd_driver.sch (KiCad schematic (older format))
At the start: 23 parts, among them J1 INPUT, J2 FIL, J3 HV, U1 LM4871, U2 LT1073CS

Commit message: add a protecting diode to the power input. make sure the right thing are pushed.
Parts:
- removed C2: 100u/63v, Capacitor_THT:CP_Radial_D8.0mm_P5.00mm, symbol Device:CP
- removed C6: 4n7, Capacitor_SMD:C_0805_2012Metric_Pad1.15x1.40mm_HandSolder, symbol Device:C
- removed C7: 1u, Capacitor_THT:C_Rect_L7.0mm_W2.0mm_P5.00mm, symbol Device:C
- removed D1: SS14, Diode_SMD:D_SMA_Handsoldering, symbol Device:D_Schottky
- removed J1: INPUT, Connector_PinHeader_2.54mm:PinHeader_1x03_P2.54mm_Vertical, symbol Connector_Generic:Conn_01x03
- removed J2: FIL, Connector_PinHeader_2.54mm:PinHeader_1x02_P2.54mm_Vertical, symbol Connector_Generic:Conn_01x02
- removed L1: 330, Choke_SMD:Choke_CD75, symbol Device:L
- removed R15, R3: 22k, Resistor_SMD:R_0805_2012Metric_Pad1.15x1.40mm_HandSolder, symbol Device:R_Small
- removed R16, R17: 18, Resistor_SMD:R_1206_3216Metric_Pad1.42x1.75mm_HandSolder, symbol Device:R
- removed R4: 10k, Resistor_SMD:R_0805_2012Metric_Pad1.15x1.40mm_HandSolder, symbol Device:R_Small
- removed U1: LM4871, Package_SO:SOIC-8_3.9x4.9mm_P1.27mm, symbol vfd_driver-rescue:LM4871-LM4871
- removed U2: LT1073CS, Package_SO:SOIC-8_3.9x4.9mm_P1.27mm, symbol Regulator_Switching:LT1073CS
- added C2: 100n, Capacitor_SMD:C_0805_2012Metric_Pad1.15x1.40mm_HandSolder, symbol Device:C
- added D1: SD103BW, Diode_SMD:D_SOD-123, symbol Device:D_Schottky_Small
- added J1: Input, Connector_PinSocket_2.54mm:PinSocket_1x07_P2.54mm_Vertical, symbol Connector_Generic:Conn_01x07
- added J2: futaba_7_lt_44z, Connector_PinSocket_2.54mm:PinSocket_1x34_P2.54mm_Vertical, symbol vfd_driver-rescue:futaba_7_lt_44z-custom-vfd_driver-rescue
- added J4: FIL_n, Connector_Pin:Pin_D1.4mm_L8.5mm_W2.8mm_FlatFork, symbol Connector_Generic:Conn_01x01
- added J5: FIL_p, Connector_Pin:Pin_D1.4mm_L8.5mm_W2.8mm_FlatFork, symbol Connector_Generic:Conn_01x01
- added L2: 33, Inductor_SMD:L_1206_3216Metric_Pad1.42x1.75mm_HandSolder, symbol Device:L_Small
- added Q3, Q5: BC817, Package_TO_SOT_SMD:SOT-23, symbol Transistor_BJT:BC817
- added Q4, Q6: BC807, Package_TO_SOT_SMD:SOT-23, symbol Transistor_BJT:BC807
- added R10, R7, R8: 33k, Resistor_SMD:R_0805_2012Metric_Pad1.15x1.40mm_HandSolder, symbol Device:R
- added R12, R13: 0, Resistor_SMD:R_1206_3216Metric, symbol Device:R
- added R6, R9: 100k, Resistor_SMD:R_0805_2012Metric_Pad1.15x1.40mm_HandSolder, symbol Device:R
- added U1, U2, U3, U4: 74HC595, Package_SO:SOIC-16_3.9x9.9mm_P1.27mm, symbol 74xx:74HC595
- added U5, U6, U7: TBD62783A, Package_SO:SOP-18_7.0x12.5mm_P1.27mm, symbol Transistor_Array:TBD62783A
- C1: value 100u -> 10u; footprint Capacitor_Tantalum_SMD:CP_EIA-7343-15_Kemet-W_Pad2.25x2.55mm_HandSolder -> Capacitor_THT:CP_Radial_D8.0mm_P3.80mm
- C5: value 100n -> 10n
- J3: value HV -> High Volt
- R1: value 50 -> 0; footprint Resistor_SMD:R_0805_2012Metric_Pad1.15x1.40mm_HandSolder -> Resistor_SMD:R_1206_3216Metric
- R2: value 1M -> 0; footprint Resistor_SMD:R_0805_2012Metric_Pad1.15x1.40mm_HandSolder -> Resistor_SMD:R_1206_3216Metric
- R5: value 10k -> 33k
Connections:
- net labels added: DATA, G1, G2, G3, G4, G5, G6, G7, Q0, Q1, Q1A, Q1B, Q1C, Q1D, Q1E, Q1F, Q1G, Q1H, Q2, Q2A, Q2B, Q2C, Q2D, Q2E, Q2F, Q2G, Q2H, Q3A, Q3B, Q3C, Q3D, Q3E, Q3F, Q3G, Q3H, Q4A, Q4B, Q4C, Q4D, Q4E, Q4F, Q4G, Q4H, RCLK, S1, S10, S11, S12, S2, S3, S4, S5, S6, S7, S8, S9, SRCLK, VCC, VDD, a, b, c, d, e, f, g, ~SRCLR
- net labels removed: +12V, +5V, FIL_n, FIL_p
- wire segments 80 -> 233
- no-connect marks 2 -> 11
Other:
- moved on the sheet: C3, C5, H1, H2

Commit message: remove unconnected wires
Parts:
- J2: symbol vfd_driver-rescue:futaba_7_lt_44z-custom-vfd_driver-rescue -> vfd_driver-rescue:futaba_7_lt_44z-custom-vfd_driver-rescue-vfd_driver-rescue
Changed lines of the file:
@@
 	5650 2100 5650 2400
 $Comp
-L vfd_driver-rescue:futaba_7_lt_44z-custom-vfd_driver-rescue J2
+L vfd_driver-rescue:futaba_7_lt_44z-custom-vfd_driver-rescue-vfd_driver-rescue J2
 U 1 1 5C057512
 P 10550 4600
@@
 	1150 1500 1300 1500
 Connection ~ 1300 1500
-Wire Wire Line
-	8600 3400 8600 3550
-Wire Wire Line
-	7850 3400 8600 3400
 $EndSCHEMATC
