File: vfd_driver.sch (KiCad schematic (older format))
At the start: 34 parts, among them J1 Input, J2 futaba_7_lt_44z, J3 High Volt, J4 FIL_n, J5 FIL_p, Q3 BC817, Q4 BC807, Q5 BC817, Q6 BC807, U1 74HC595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

Commit message: remove resistor and align comments
Parts:
- removed R1, R12, R13, R2: 0, Resistor_SMD:R_1206_3216Metric, symbol Device:R
Changed lines of the file:
@@
 $EndComp
-$Comp
-L power:+36V #PWR03
-U 1 1 5C6D1A84
-P 1100 5300
-F 0 "#PWR03" H 1100 5150 50  0001 C CNN
-F 1 "+36V" H 1115 5473 50  0000 C CNN
-F 2 "" H 1100 5300 50  0001 C CNN
-F 3 "" H 1100 5300 50  0001 C CNN
-	1    1100 5300
-	1    0    0    -1
-$EndComp
-$Comp
-L power:+36V #PWR04
-U 1 1 5C6D1B07
-P 1700 5300
-F 0 "#PWR04" H 1700 5150 50  0001 C CNN
-F 1 "+36V" H 1715 5473 50  0000 C CNN
-F 2 "" H 1700 5300 50  0001 C CNN
-F 3 "" H 1700 5300 50  0001 C CNN
-	1    1700 5300
-	1    0    0    -1
-$EndComp
-$Comp
-L Device:R R12
-U 1 1 5C6D1B62
-P 1400 5400
-F 0 "R12" V 1300 5350 50  0000 L CNN
-F 1 "0" V 1400 5400 50  0000 L CNN
-F 2 "Resistor_SMD:R_1206_3216Metric" V 1330 5400 50  0001 C CNN
-F 3 "~" H 1400 5400 50  0001 C CNN
-	1    1400 5400
-	0    1    1    0
-$EndComp
-Wire Wire Line
-	1550 5400 1700 5400
-Wire Wire Line
-	1700 5400 1700 5300
-Wire Wire Line
-	1250 5400 1100 5400
-Wire Wire Line
-	1100 5400 1100 5300
-$Comp
-L Device:R R13
-U 1 1 5C70AD81
-P 1400 5600
-F 0 "R13" V 1300 5550 50  0000 L CNN
-F 1 "0" V 1400 5600 50  0000 L CNN
-F 2 "Resistor_SMD:R_1206_3216Metric" V 1330 5600 50  0001 C CNN
-F 3 "~" H 1400 5600 50  0001 C CNN
-	1    1400 5600
-	0    1    1    0
-$EndComp
-Wire Wire Line
-	1550 5600 1700 5600
-Wire Wire Line
-	1700 5600 1700 5400
-Connection ~ 1700 5400
-Wire Wire Line
-	1250 5600 1100 5600
-Wire Wire Line
-	1100 5600 1100 5400
-Connection ~ 1100 5400
 $Comp
 L Device:L_Small L2
@@
 Wire Wire Line
 	1550 6400 1550 6150
-$Comp
-L Device:R R1
-U 1 1 5CB52232
-P 1400 7200
-F 0 "R1" V 1300 7150 50  0000 L CNN
-F 1 "0" V 1400 7200 50  0000 L CNN
-F 2 "Resistor_SMD:R_1206_3216Metric" V 1330 7200 50  0001 C CNN
-F 3 "~" H 1400 7200 50  0001 C CNN
-	1    1400 7200
-	0    1    1    0
-$EndComp
-Wire Wire Line
-	1550 7200 1700 7200
-Wire Wire Line
-	1250 7200 1100 7200
-$Comp
-L Device:R R2
-U 1 1 5CB5223D
-P 1400 7400
-F 0 "R2" V 1300 7350 50  0000 L CNN
-F 1 "0" V 1400 7400 50  0000 L CNN
-F 2 "Resistor_SMD:R_1206_3216Metric" V 1330 7400 50  0001 C CNN
-F 3 "~" H 1400 7400 50  0001 C CNN
-	1    1400 7400
-	0    1    1    0
-$EndComp
-Wire Wire Line
-	1550 7400 1700 7400
-Wire Wire Line
-	1700 7400 1700 7200
-Connection ~ 1700 7200
-Wire Wire Line
-	1250 7400 1100 7400
-Wire Wire Line
-	1100 7400 1100 7200
-Connection ~ 1100 7200
-Text Label 1300 7000 0    50   ~ 0
-SRCLK
-Wire Wire Line
-	1100 7000 1700 7000
-Wire Wire Line
-	1700 7000 1700 7200
-Wire Wire Line
-	1100 7000 1100 7200
 Wire Wire Line
 	1700 3500 1700 3700

Commit message: arranging labels
Parts:
- J2: symbol vfd_driver-rescue:futaba_7_lt_44z-custom-vfd_driver-rescue -> vfd_driver-rescue:futaba_7_lt_44z-custom-vfd_driver-rescue-vfd_driver-rescue
Changed lines of the file:
@@
 	5650 2100 5650 2400
 $Comp
-L vfd_driver-rescue:futaba_7_lt_44z-custom-vfd_driver-rescue J2
+L vfd_driver-rescue:futaba_7_lt_44z-custom-vfd_driver-rescue-vfd_driver-rescue J2
 U 1 1 5C057512
 P 10550 4600
